File: hardware/v0/esp32_sensor_board/wrong_esp32_sensor_board.kicad_pcb (KiCad board)
At the start: 4 copper layers, 76 x 62 mm, 86 parts, among them J101 Conn_01x02, J102 Conn_01x02, J103 Conn_01x02, J104 Conn_01x02, J201 3.3V, J301 USB_B_Micro, J302 Micro_SD_Card_Det, J303 Conn_Coaxial, J304 UART, J305 EXT1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

Commit message: WIP
Parts:
- removed C315: 0.1uF, Capacitor_SMD:C_0603_1608Metric
- removed G***: LOGO, BVH_Logos:SkyIron_logo_Back
- removed R307, R308, R309, R310: 50k, Resistor_SMD:R_0603_1608Metric
- removed U303: ~, BVH_Components_Misc:Diode_10Pin_DFN2510A-10_10-XFDFN_SOT1176-1
- moved J307 67.3 mm to (87.5, 83.7), turned to 0 degrees
- moved J305 5.34 mm to (148.6, 104.5), turned to -90 degrees
- moved J306 5.03 mm to (148.5, 100.5), turned to -90 degrees
- moved C307 1.28 mm to (111.2, 93.0)
- moved L301 1.28 mm to (110.7, 94.5)
- moved SW302 1.27 mm to (109.6, 71.9)
- moved C302 1.00 mm to (118.5, 99.5)
- moved C301 0.55 mm to (120.5, 100.0)
- moved SW301 0.34 mm to (136.0, 98.0)
- moved J308 0.14 mm to (131.0, 93.0)
Connections:
- J302 pad 4: Net-(J302-VDD) -> +3.3V
Routing:
- net /Load Cell Sensor/DRDY_NAU: track 38.0 -> 0.00 mm, vias 2 -> 0
- net /Microprocessor/SPI_SCK: track 42.9 -> 27.0 mm
- net /Power Measurement/I2C_SCL: track 126.9 -> 113.2 mm, vias 6 -> 5
- net /Microprocessor/SPI_COPI: track 43.6 -> 30.9 mm
- net Net-(J302-VDD): track 9.49 -> 0.00 mm, vias 2 -> 0
- net +3.3V: track 71.4 -> 62.6 mm, vias 30 -> 28
- net /Power Measurement/I2C_SDA: track 125.4 -> 116.7 mm
- net /Microprocessor/SPI_CIPO: track 39.2 -> 31.1 mm
- net GND: track 83.2 -> 75.5 mm, vias 68 -> 66
- net /Microprocessor/EXT_1: track 37.8 -> 31.3 mm
- net /Microprocessor/EXT_2: track 30.5 -> 24.4 mm
- net /Microprocessor/SPI_CS1: track 28.9 -> 22.9 mm
- net /Microprocessor/SD_CS: track 23.1 -> 20.6 mm
- net /Microprocessor/VDD33A: track 5.57 -> 6.85 mm
- net /Microprocessor/STATUS_LED: track 11.1 -> 10.1 mm
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Other:
- board text added: "DO NOT CLOSE J201 WHEN J1 POWERED"
- board text removed: "+V"
- board text removed: "3.3"
- board text removed: "CTL"
- board text removed: "DO NOT CLOSE J201 WHEN USING J101"
- board text removed: "GND"
- board text removed: "PGOOD"
- board text removed: "SCL"
- board text removed: "SDA"
- board text removed: "Vin"
