File: hardware/v0/esp32_sensor_board/esp32_uc.kicad_sch (KiCad schematic)
At the start: 43 parts, among them J301 USB_B_Micro, J302 Micro_SD_Card_Det, J303 Conn_Coaxial, J304 UART, J305 EXT1, J306 EXT2, J307 I2C, J308 SPI, SW301 SW_SPST, SW302 RST, U302 ESP32-C3, Y301 32kHz RTC Crystal, Y302 40 MHz

Commit message: Relay board, firmware tests
Parts:
- C313, C314: value C_Small -> 2.1pF
- L302: value L_Small -> 5.6nH
Changed lines of the file:
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@@
     (effects (font (size 1.27 1.27)) (justify left bottom))
   )
-  (text "Power Filtering" (at 17.78 17.78 0)
+  (text "Power Filtering" (at 34.29 17.78 0)
     (effects (font (size 1.27 1.27)) (justify left bottom))
   )
@@
     (effects (font (size 1.27 1.27)) (justify right bottom))
   )
-  (label "RF_ANT" (at 41.91 140.97 0) (fields_autoplaced)
+  (label "RF_ANT" (at 45.72 140.97 0) (fields_autoplaced)
     (effects (font (size 1.27 1.27)) (justify left bottom))
   )
@@
       (effects (font (size 1.27 1.27)) (justify left))
     )
-    (property "Value" "C_Small" (at 46.99 147.3263 0)
+    (property "Value" "2.1pF" (at 46.99 147.3263 0)
       (effects (font (size 1.27 1.27)) (justify left))
     )
@@
       (effects (font (size 1.27 1.27)) (justify left))
     )
-    (property "Value" "C_Small" (at 26.67 147.3263 0)
+    (property "Value" "2.1pF" (at 26.67 147.3263 0)
       (effects (font (size 1.27 1.27)) (justify left))
     )
@@
       (effects (font (size 1.27 1.27)))
     )
-    (property "Value" "L_Small" (at 34.29 138.43 90)
-      (effects (font (size 1.27 1.27)))
-    )
+    (property "Value" "5.6nH" (at 34.29 138.43 90)
+      (effects (font (size 1.27 1.27)))
+    )

Commit message: WIP v3 hardware
Parts:
- removed J301: USB_B_Micro, Connector_USB:USB_Micro-B_Molex-105017-0001, symbol Connector:USB_B_Micro
- added J301: USB4510-03-1-A_REVA, USB4510-03-1-A_REVA:GCT_USB4510-03-1-A_REVA, symbol USB4510-03-1-A:USB4510-03-1-A_REVA
- added R311, R312: 5.1k, Resistor_SMD:R_0603_1608Metric, symbol Device:R_Small
- SW301: value SW_SPST -> BOOT
Connections:
- net +5V: now also J301.A4_B9 (VBUS_A), J301.B4_A9 (VBUS_B)
- net GND: now also J301.A1_B12 (GND_A), J301.B1_A12 (GND_B), R311.1, R312.1
- net USB_N: now also J301.A7 (DN1), J301.B7 (DN2)
- net USB_P: now also J301.A6 (DP1), J301.B6 (DP2)
- new net: J301.B5 (CC2), R312.2
- new net: J301.A5 (CC1), R311.2
- new net: J301.S1 (SHELL_GND), J301.S2 (SHELL_GND), J301.S3 (SHELL_GND), J301.S4 (SHELL_GND)
- no-connect marks 4 -> 5
Other:
- moved on the sheet: J304, J305, J306, J307, U301
