File: hardware/v0/esp32_sensor_board/esp32_uc.kicad_sch (KiCad schematic)
At the start: 45 parts, among them J301 USB4510-03-1-A_REVA, J302 Micro_SD_Card_Det, J303 Conn_Coaxial, J304 UART, J305 EXT1, J306 EXT2, J307 I2C, J308 SPI, SW301 BOOT, SW302 RST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

Commit message: WIP
Parts:
- J301: footprint USB4510-03-1-A_REVA:GCT_USB4510-03-1-A_REVA -> USB4510-03-1-A:GCT_USB4510-03-1-A_REVA
Connections:
- net +3.3V: now also C315.2, J302.4 (VDD); no longer C315.1
- net GND: now also C315.1
- net SPI_CIPO: now also U303.4 (CH3); no longer U303.1 (CH1)
- net SPI_SCK: now also U303.1 (CH1); no longer U303.4 (CH3)
Other:
- moved on the sheet: C315
Changed lines of the file:
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@@
 	)
 	(junction
+		(at 217.17 135.89)
+		(diameter 0)
+		(color 0 0 0 0)
+	)
+	(junction
 		(at 74.93 160.02)
 		(diameter 0)
@@
 	)
 	(junction
-		(at 240.03 146.05)
-		(diameter 0)
-		(color 0 0 0 0)
-	)
-	(junction
 		(at 278.13 105.41)
 		(diameter 0)
@@
 	)
 	(junction
+		(at 219.71 140.97)
+		(diameter 0)
+		(color 0 0 0 0)
+	)
+	(junction
 		(at 219.71 156.21)
 		(diameter 0)
@@
 	(wire
 		(pts
-			(xy 219.71 138.43) (xy 219.71 149.86)
+			(xy 219.71 138.43) (xy 219.71 140.97)
 		)
 		(stroke
@@
 	(wire
 		(pts
-			(xy 227.33 135.89) (xy 226.06 135.89)
-		)
-		(stroke
-			(width 0)
-			(type default)
-		)
-	)
-	(wire
-		(pts
 			(xy 101.6 124.46) (xy 106.68 124.46)
 		)
@@
 	(wire
 		(pts
-			(xy 217.17 135.89) (xy 220.98 135.89)
+			(xy 217.17 135.89) (xy 227.33 135.89)
 		)
 		(stroke
@@
 	(wire
 		(pts
+			(xy 219.71 140.97) (xy 219.71 149.86)
+		)
+		(stroke
+			(width 0)
+			(type default)
+		)
+	)
+	(wire
+		(pts
 			(xy 237.49 143.51) (xy 240.03 143.51)
 		)
@@
 		)
 	)
-	(bus
+	(wire
 		(pts
-			(xy 12.7 160.02) (xy 74.93 160.02)
+			(xy 227.33 146.05) (xy 240.03 146.05)
 		)
 		(stroke
@@
 		)
 	)
-	(wire
+	(bus
 		(pts
-			(xy 242.57 146.05) (xy 240.03 146.05)
+			(xy 12.7 160.02) (xy 74.93 160.02)
 		)
 		(stroke
@@
 	(wire
 		(pts
+			(xy 215.9 135.89) (xy 217.17 135.89)
+		)
+		(stroke
+			(width 0)
+			(type default)
+		)
+	)
+	(wire
+		(pts
 			(xy 267.97 120.65) (xy 270.51 120.65)
 		)
@@
 	(wire
 		(pts
-			(xy 233.68 114.3) (xy 237.49 114.3)
+			(xy 215.9 140.97) (xy 219.71 140.97)
 		)
 		(stroke
@@
 	(wire
 		(pts
-			(xy 223.52 96.52) (xy 223.52 101.6)
+			(xy 233.68 114.3) (xy 237.49 114.3)
 		)
 		(stroke
@@
 	(wire
 		(pts
-			(xy 275.59 120.65) (xy 278.13 120.65)
+			(xy 223.52 96.52) (xy 223.52 101.6)
 		)
 		(stroke
@@
 	(wire
 		(pts
-			(xy 227.33 146.05) (xy 240.03 146.05)
+			(xy 275.59 120.65) (xy 278.13 120.65)
 		)
 		(stroke
@@
 	)
 	(label "SPI_CIPO"
-		(at 181.61 134.62 180)
+		(at 181.61 142.24 180)
 		(fields_autoplaced yes)
 		(effects
@@
 	)
 	(label "SPI_SCK"
-		(at 181.61 142.24 180)
+		(at 181.61 134.62 180)
 		(fields_autoplaced yes)
 		(effects
@@
 	(symbol
 		(lib_id "Device:C_Small")
-		(at 223.52 135.89 90)
+		(at 215.9 138.43 180)
 		(unit 1)
 		(exclude_from_sim no)
@@
 		(on_board yes)
 		(dnp no)
-		(fields_autoplaced yes)
 		(property "Reference" "C315"
-			(at 223.5263 129.54 90)
+			(at 213.36 142.748 0)
 			(effects
 				(font
 					(size 1.27 1.27)
 				)
+				(justify right)
 			)
 		)
 		(property "Value" "0.1uF"
-			(at 223.5263 132.08 90)
+			(at 213.106 144.78 0)
 			(effects
 				(font
 					(size 1.27 1.27)
 				)
+				(justify right)
 			)
 		)
 		(property "Footprint" "Capacitor_SMD:C_0603_1608Metric"
-			(at 223.52 135.89 0)
+			(at 215.9 138.43 0)
 			(effects
 				(font
@@
 		)
 		(property "Datasheet" "~"
-			(at 223.52 135.89 0)
+			(at 215.9 138.43 0)
 			(effects
 				(font
@@
 		)
 		(property "Description" ""
-			(at 223.52 135.89 0)
+			(at 215.9 138.43 0)
 			(effects
 				(font
@@
 			)
 		)
-		(property "Footprint" "USB4510-03-1-A_REVA:GCT_USB4510-03-1-A_REVA"
+		(property "Footprint" "USB4510-03-1-A:GCT_USB4510-03-1-A_REVA"
 			(at 245.11 73.66 0)
 			(effects

Commit message: Output files
Parts:
- added R313: 33R, symbol Device:R_Small
- added R314: 50k, Resistor_SMD:R_0603_1608Metric, symbol Device:R_Small
Connections:
- net +3.3V: now also R313.1, R314.1; no longer J302.4 (VDD)
- net GND: no longer J302.1 (DAT2)
- new net: J302.4 (VDD), R313.2
- new net SD_DAT2: J302.1 (DAT2), R314.2
Other:
- moved on the sheet: R307, R308, R309, R310

Commit message: Revisions for recordering
Parts:
- removed J301: USB4510-03-1-A_REVA, USB4510-03-1-A:GCT_USB4510-03-1-A_REVA, symbol USB4510-03-1-A:USB4510-03-1-A_REVA
- added J309: USB_C_Receptacle_USB2.0_16P, Connector_USB:USB_C_Receptacle_GCT_USB4085, symbol Connector:USB_C_Receptacle_USB2.0_16P
- R313: footprint (none) -> Resistor_SMD:R_0603_1608Metric
Connections:
- net +5V: now also J309.A4 (VBUS), J309.A9 (VBUS), J309.B4 (VBUS), J309.B9 (VBUS)
- net GND: now also J309.A1 (GND), J309.A12 (GND), J309.B1 (GND), J309.B12 (GND)
- net USB_N: now also J309.A7 (D-), J309.B7 (D-)
- net USB_P: now also J309.A6 (D+), J309.B6 (D+)
- net at R312.2: now also J309.B5 (CC2)
- net at R311.2: now also J309.A5 (CC1)
Other:
- moved on the sheet: R311, R312
