File: hardware/v0/esp32_sensor_board/esp32_sensor_power.kicad_sch (KiCad schematic)
At the start: 13 parts, among them U202 LMR36006

Commit message: Clean up errors
Other:
- moved on the sheet: C202, C204, C205, C206, R202, R204

Commit message: PCB ordered, a few initial mistakes fixed
Parts:
- added JP201: Jumper_2_Open, Jumper:SolderJumper-2_P1.3mm_Open_RoundedPad1.0x1.5mm, symbol Jumper:Jumper_2_Open
- U201: renamed from U202; footprint Package_SO:Texas_HSOP-8-1EP_3.9x4.9mm_P1.27mm_ThermalVias -> BVH_Power:LMR36006-VQFN-HR
- renumbered C205 to C201, C201 to C202, C207 to C205, C208 to C206, C206 to C207, C202 to C208, R204 to R203
Connections:
- net GND: now also U201.11 (PGND)
- net VCC: now reaches C208.1, U201.5 (VCC)
- net FB: now reaches C207.2, R201.2, R202.1, U201.7 (FB)
- net at C201.1: now also U201.4 (BOOT); no longer U201.11 (BOOT)
- net SW: now reaches C201.2, L201.1, U201.12 (SW)
- net SW: now also U201.3 (SW)
- net +48V renamed VIN
- net VIN: now also JP201.2 (B)
- new net +5V: JP201.1 (A)
Other:
- note added: "Discarded options"
- note added: "LMR36006-Q1 - 4.2V - 60V input - Integrated FET - 3.3V, 5V fixed or Adjustable output - Power Good signal - $2.71 in single quantities LMR36006CRNXT - Adjustable, 2.1 MHz switching frequency"
- note added: "Optional USB power input. Unprotected, do not use with external power."
- note removed: "LMR36006-Q1 - 4.2V - 60V input - Integrated FET - 3.3V, 5V fixed or Adjustable output - Power Good signal LMR36006CRNXT - Adjustable, 2.1 MHz switching frequency"

Commit message: Board refactor WIP.  Still needs PU resistors
Parts:
- added J201: 3.3V, Connector_PinHeader_2.54mm:PinHeader_1x03_P2.54mm_Vertical, symbol Connector:Conn_01x03_Socket
Connections:
- net +3.3V: now also J201.2 (Pin_2)
- net GND: now also J201.1 (Pin_1)
- net P_GOOD: now also J201.3 (Pin_3)
Changed lines of the file:
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@@
+    (stroke (width 0) (type default))
+  )
+  (wire (pts (xy 54.61 132.08) (xy 57.15 132.08))
+    (stroke (width 0) (type default))
+  )
+  (wire (pts (xy 77.47 172.72) (xy 77.47 177.8))
     (stroke (width 0) (type default))
   )
@@
     (stroke (width 0) (type default))
   )
+  (wire (pts (xy 54.61 129.54) (xy 57.15 129.54))
+    (stroke (width 0) (type default))
+  )
   (wire (pts (xy 139.7 58.42) (xy 149.86 58.42))
     (stroke (width 0) (type default))
@@
     (stroke (width 0) (type default))
   )
+  (wire (pts (xy 54.61 139.7) (xy 57.15 139.7))
+    (stroke (width 0) (type default))
+  )
   (wire (pts (xy 68.58 35.56) (xy 76.2 35.56))
     (stroke (width 0) (type default))
@@
     (stroke (width 0) (type default))
   )
+  (wire (pts (xy 54.61 137.16) (xy 54.61 132.08))
+    (stroke (width 0) (type default))
+  )
   (wire (pts (xy 58.42 55.88) (xy 66.04 55.88))
     (stroke (width 0) (type default))
   )
+  (wire (pts (xy 57.15 139.7) (xy 57.15 134.62))
+    (stroke (width 0) (type default))
+  )
   (wire (pts (xy 58.42 35.56) (xy 53.34 35.56))
     (stroke (width 0) (type default))
@@
     (stroke (width 0) (type default))
   )
+  (wire (pts (xy 49.53 137.16) (xy 54.61 137.16))
+    (stroke (width 0) (type default))
+  )
   (wire (pts (xy 177.8 86.36) (xy 180.34 86.36))
     (stroke (width 0) (type default))
@@
     (stroke (width 0) (type default))
   )
+  (wire (pts (xy 49.53 123.19) (xy 54.61 123.19))
+    (stroke (width 0) (type default))
+  )
   (wire (pts (xy 53.34 35.56) (xy 53.34 30.48))
     (stroke (width 0) (type default))
@@
     (stroke (width 0) (type default))
   )
+  (wire (pts (xy 54.61 123.19) (xy 54.61 129.54))
+    (stroke (width 0) (type default))
+  )
   (wire (pts (xy 78.74 73.66) (xy 78.74 76.2))
     (stroke (width 0) (type default))
@@
     (stroke (width 0) (type default))
   )
-  (wire (pts (xy 25.4 35.56) (xy 25.4 40.64))
+  (wire (pts (xy 57.15 172.72) (xy 57.15 177.8))
     (stroke (width 0) (type default))
   )
@@
   (label "VCC" (at 63.5 66.04 0) (fields_autoplaced)
     (effects (font (size 1.27 1.27)) (justify left bottom))
+  )
+  (global_label "P_GOOD" (shape input) (at 54.61 139.7 180) (fields_autoplaced)
+    (effects (font (size 1.27 1.27)) (justify right))
+    (property "Intersheetrefs" "${INTERSHEET_REFS}" (at 44.1862 139.7 0)
+      (effects (font (size 1.27 1.27)) (justify right) hide)
+    )
   )
   (global_label "P_GOOD" (shape input) (at 91.44 66.04 0) (fields_autoplaced)
@@
     )
   )
-  (hierarchical_label "PWR_IN" (shape input) (at 25.4 35.56 180) (fields_autoplaced)
+  (hierarchical_label "PWR_IN" (shape input) (at 57.15 172.72 180) (fields_autoplaced)
     (effects (font (size 1.27 1.27)) (justify right))
   )
@@
     )
   )
+  (symbol (lib_id "power:+3.3V") (at 49.53 137.16 0) (unit 1)
+    (in_bom yes) (on_board yes) (dnp no)
+    (property "Reference" "#PWR0202" (at 49.53 140.97 0)
+      (effects (font (size 1.27 1.27)) hide)
+    )
+    (property "Value" "+3.3V" (at 49.53 132.08 0)
+      (effects (font (size 1.27 1.27)))
+    )
+    (property "Footprint" "" (at 49.53 137.16 0)
+      (effects (font (size 1.27 1.27)) hide)
+    )
+    (property "Datasheet" "" (at 49.53 137.16 0)
+      (effects (font (size 1.27 1.27)) hide)
+    )
+    (pin "1")
+    (instances
+      (project "esp32_sensor_board"
+        (path "/d76badc5-1f0d-4fe6-889f-ca56408e093d/1fe32be5-ab10-4126-a012-3b12c483f6b3"
+          (reference "#PWR0202") (unit 1)
+        )
+      )
+    )
+  )
   (symbol (lib_id "power:GND") (at 124.46 83.82 0) (unit 1)
     (in_bom yes) (on_board yes) (dnp no) (fields_autoplaced)
@@
         (path "/d76badc5-1f0d-4fe6-889f-ca56408e093d/1fe32be5-ab10-4126-a012-3b12c483f6b3"
           (reference "#PWR0209") (unit 1)
+        )
+      )
+    )
+  )
+  (symbol (lib_id "power:GND") (at 49.53 123.19 0) (unit 1)
+    (in_bom yes) (on_board yes) (dnp no)
+    (property "Reference" "#PWR0210" (at 49.53 129.54 0)
+      (effects (font (size 1.27 1.27)) hide)
+    )
+    (property "Value" "GND" (at 49.53 128.27 0)
+      (effects (font (size 1.27 1.27)))
+    )
+    (property "Footprint" "" (at 49.53 123.19 0)
+      (effects (font (size 1.27 1.27)) hide)
+    )
+    (property "Datasheet" "" (at 49.53 123.19 0)
+      (effects (font (size 1.27 1.27)) hide)
+    )
+    (pin "1")
+    (instances
+      (project "esp32_sensor_board"
+        (path "/d76badc5-1f0d-4fe6-889f-ca56408e093d/1fe32be5-ab10-4126-a012-3b12c483f6b3"
+          (reference "#PWR0210") (unit 1)
         )
       )
@@
     )
   )
-  (symbol (lib_id "power:PWR_FLAG") (at 25.4 40.64 180) (unit 1)
-    (in_bom yes) (on_board yes) (dnp no) (fields_autoplaced)
-    (property "Reference" "#FLG0201" (at 25.4 42.545 0)
-      (effects (font (size 1.27 1.27)) hide)
-    )
-    (property "Value" "PWR_FLAG" (at 25.4 45.72 0)
-      (effects (font (size 1.27 1.27)))
-    )
-    (property "Footprint" "" (at 25.4 40.64 0)
-      (effects (font (size 1.27 1.27)) hide)
-    )
-    (property "Datasheet" "~" (at 25.4 40.64 0)
+  (symbol (lib_id "power:PWR_FLAG") (at 57.15 177.8 180) (unit 1)
+    (in_bom yes) (on_board yes) (dnp no) (fields_autoplaced)
+    (property "Reference" "#FLG0201" (at 57.15 179.705 0)
+      (effects (font (size 1.27 1.27)) hide)
+    )
+    (property "Value" "PWR_FLAG" (at 57.15 182.88 0)
+      (effects (font (size 1.27 1.27)))
+    )
+    (property "Footprint" "" (at 57.15 177.8 0)
+      (effects (font (size 1.27 1.27)) hide)
+    )
+    (property "Datasheet" "~" (at 57.15 177.8 0)
       (effects (font (size 1.27 1.27)) hide)
     )
@@
         (path "/d76badc5-1f0d-4fe6-889f-ca56408e093d/1fe32be5-ab10-4126-a012-3b12c483f6b3"
           (reference "R201") (unit 1)
+        )
+      )
+    )
+  )
+  (symbol (lib_id "Connector:Conn_01x03_Socket") (at 62.23 132.08 0) (unit 1)
+    (in_bom yes) (on_board yes) (dnp no) (fields_autoplaced)
+    (property "Reference" "J201" (at 63.5 132.08 0)
+      (effects (font (size 1.27 1.27)) (justify left))
+    )
+    (property "Value" "3.3V" (at 63.5 134.62 0)
+      (effects (font (size 1.27 1.27)) (justify left))
+    )
+    (property "Footprint" "Connector_PinHeader_2.54mm:PinHeader_1x03_P2.54mm_Vertical" (at 62.23 132.08 0)
+      (effects (font (size 1.27 1.27)) hide)
+    )
+    (property "Datasheet" "~" (at 62.23 132.08 0)
+      (effects (font (size 1.27 1.27)) hide)
+    )
+    (pin "1")
+    (pin "2")
+    (pin "3")
+    (instances
+      (project "esp32_sensor_board"
+        (path "/d76badc5-1f0d-4fe6-889f-ca56408e093d/1fe32be5-ab10-4126-a012-3b12c483f6b3"
+          (reference "J201") (unit 1)
         )
       )
@@
     )
   )
+  (symbol (lib_id "power:+3.3V") (at 77.47 172.72 0) (unit 1)
+    (in_bom yes) (on_board yes) (dnp no) (fields_autoplaced)
+    (property "Reference" "#PWR0211" (at 77.47 176.53 0)
+      (effects (font (size 1.27 1.27)) hide)
+    )
+    (property "Value" "+3.3V" (at 77.47 167.64 0)
+      (effects (font (size 1.27 1.27)))
+    )
+    (property "Footprint" "" (at 77.47 172.72 0)
+      (effects (font (size 1.27 1.27)) hide)
+    )
+    (property "Datasheet" "" (at 77.47 172.72 0)
+      (effects (font (size 1.27 1.27)) hide)
+    )
+    (pin "1")
+    (instances
+      (project "esp32_sensor_board"
+        (path "/d76badc5-1f0d-4fe6-889f-ca56408e093d/1fe32be5-ab10-4126-a012-3b12c483f6b3"
+          (reference "#PWR0211") (unit 1)
+        )
+      )
+    )
+  )
   (symbol (lib_id "Device:L_Small") (at 111.76 58.42 90) (unit 1)
     (in_bom yes) (on_board yes) (dnp no) (fields_autoplaced)
@@
         )
       )
+    )
+  )
+  (symbol (lib_id "power:PWR_FLAG") (at 77.47 177.8 180) (unit 1)
+    (in_bom yes) (on_board yes) (dnp no) (fields_autoplaced)
+    (property "Reference" "#FLG0202" (at 77.47 179.705 0)
+      (effects (font (size 1.27 1.27)) hide)
+    )
+    (property "Value" "PWR_FLAG" (at 77.47 182.88 0)
+      (effects (font (size 1.27 1.27)))
+    )
+    (property "Footprint" "" (at 77.47 177.8 0)
+      (effects (font (size 1.27 1.27)) hide)
+    )
+    (property "Datasheet" "~" (at 77.47 177.8 0)
+      (effects (font (size 1.27 1.27)) hide)
+    )
+    (pin "1")
+    (instances
+      (project "esp32_sensor_board"
+        (path "/d76badc5-1f0d-4fe6-889f-ca56408e093d/1fe32be5-ab10-4126-a012-3b12c483f6b3"
+          (reference "#FLG0202") (unit 1)
+        )
+      )

Commit message: WIP v3 hardware
Parts:
- added D1: D_Small, symbol Device:D_Small
- JP201: value Jumper_2_Open -> USB Power Jumper; footprint Jumper:SolderJumper-2_P1.3mm_Open_RoundedPad1.0x1.5mm -> Jumper:SolderJumper-2_P1.3mm_Bridged_RoundedPad1.0x1.5mm; symbol Jumper:Jumper_2_Open -> Jumper:Jumper_2_Bridged
Connections:
- net VIN: now also D1.1 (K); no longer JP201.2 (B)
- new net: D1.2 (A), JP201.2 (B)
Other:
- note added: "Optional USB power input. LMR36006 requires 4.2V minimum, diode drop must be less than 0.8V"
- note removed: "Optional USB power input. Unprotected, do not use with external power."
Changed lines of the file:
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@@
+	(wire
+		(pts
+			(xy 81.28 35.56) (xy 88.9 35.56)
+		)
+		(stroke
+			(width 0)
+			(type default)
+		)
+	)
 	(wire
 		(pts
@@
 		)
 	)
-	(text "Optional USB power input.  \nUnprotected, do not use with external power."
+	(text "Optional USB power input.  \nLMR36006 requires 4.2V minimum, diode drop must be less than 0.8V"
 		(exclude_from_sim no)
 		(at 45.72 43.18 0)
@@
 	(hierarchical_label "PWR_IN"
 		(shape input)
-		(at 76.2 35.56 0)
+		(at 88.9 35.56 0)
 		(fields_autoplaced yes)
 		(effects
@@
 	)
 	(symbol
-		(lib_id "Jumper:Jumper_2_Open")
+		(lib_id "Jumper:Jumper_2_Bridged")
 		(at 63.5 35.56 0)
 		(unit 1)
-		(exclude_from_sim no)
+		(exclude_from_sim yes)
 		(in_bom yes)
 		(on_board yes)
@@
 		(fields_autoplaced yes)
 		(property "Reference" "JP201"
-			(at 63.5 29.21 0)
-			(effects
-				(font
-					(size 1.27 1.27)
-				)
-			)
-		)
-		(property "Value" "Jumper_2_Open"
-			(at 63.5 31.75 0)
-			(effects
-				(font
-					(size 1.27 1.27)
-				)
-			)
-		)
-		(property "Footprint" "Jumper:SolderJumper-2_P1.3mm_Open_RoundedPad1.0x1.5mm"
+			(at 63.5 30.48 0)
+			(effects
+				(font
+					(size 1.27 1.27)
+				)
+			)
+		)
+		(property "Value" "USB Power Jumper"
+			(at 63.5 33.02 0)
+			(effects
+				(font
+					(size 1.27 1.27)
+				)
+			)
+		)
+		(property "Footprint" "Jumper:SolderJumper-2_P1.3mm_Bridged_RoundedPad1.0x1.5mm"
 			(at 63.5 35.56 0)
 			(effects
@@
 			)
 		)
-		(property "Description" ""
+		(property "Description" "Jumper, 2-pole, closed/bridged"
 			(at 63.5 35.56 0)
 			(effects
@@
 					(unit 1)
 				)
+			)
+		)
+	)
+	(symbol
+		(lib_id "Device:D_Small")
+		(at 78.74 35.56 180)
+		(unit 1)
+		(exclude_from_sim no)
+		(in_bom yes)
+		(on_board yes)
+		(dnp no)
+		(fields_autoplaced yes)
+		(property "Reference" "D1"
+			(at 78.74 29.21 0)
+			(effects
+				(font
+					(size 1.27 1.27)
+				)
+			)
+		)
+		(property "Value" "D_Small"
+			(at 78.74 31.75 0)
+			(effects
+				(font
+					(size 1.27 1.27)
+				)
+			)
+		)
+		(property "Footprint" ""
+			(at 78.74 35.56 90)
+			(effects
+				(font
+					(size 1.27 1.27)
+				)
+				(hide yes)
+			)
+		)
+		(property "Datasheet" "~"
+			(at 78.74 35.56 90)
+			(effects
+				(font
+					(size 1.27 1.27)
+				)
+				(hide yes)
+			)
+		)
+		(property "Description" "Diode, small symbol"
+			(at 78.74 35.56 0)
+			(effects
+				(font
+					(size 1.27 1.27)
+				)
+				(hide yes)
+			)
+		)
+		(property "Sim.Device" "D"
+			(at 78.74 35.56 0)
+			(effects
+				(font
+					(size 1.27 1.27)
+				)
+				(hide yes)
+			)
+		)
+		(property "Sim.Pins" "1=K 2=A"
+			(at 78.74 35.56 0)
+			(effects
+				(font
+					(size 1.27 1.27)
+				)
+				(hide yes)
+			)
+		)
+		(pin "2"
+		)
+		(pin "1"
+		)
+		(instances
+			(project ""
+				(path "/d76badc5-1f0d-4fe6-889f-ca56408e093d/1fe32be5-ab10-4126-a012-3b12c483f6b3"
+					(reference "D1")
+					(unit 1)
+				)

Commit message: WIP
Parts:
- D1: footprint (none) -> Diode_SMD:D_SOD-123
Changed lines of the file:
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@@
 			)
 		)
-		(property "Footprint" ""
+		(property "Footprint" "Diode_SMD:D_SOD-123"
 			(at 78.74 35.56 90)
 			(effects
