File: hardware/v0/esp32_sensor_board/esp32_sensor_board.kicad_pcb (KiCad board)
At the start: 4 copper layers, 76 x 62 mm, 89 parts, among them J101 Conn_01x02, J102 Conn_01x02, J103 Conn_01x02, J104 Conn_01x02, J201 PWR, J301 USB4510-03-1-A_REVA, J302 Micro_SD_Card_Det, J303 Conn_Coaxial, J304 UART, J305 EXT1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

Commit message: Output files
Parts:
- added R314: 50k, Resistor_SMD:R_0603_1608Metric, F.Cu at (136.8, 79.8)
- J201: value PWR -> 3.3V
- moved G*** 20.0 mm to (111.5, 95.2)
- moved R307 1.90 mm to (136.8, 85.8), turned to 180 degrees
- moved R308 1.45 mm to (136.8, 81.2), turned to 180 degrees
- moved R310 1.38 mm to (136.8, 82.8), turned to 180 degrees
- moved R309 0.63 mm to (136.8, 84.2), turned to 180 degrees
Connections:
- J302 pad 1: GND -> /Microprocessor/SD_DAT2
- J302 pad 4: +3.3V -> Net-(J302-VDD)
Routing:
- net GND: track 85.3 -> 132.3 mm
- net /Microprocessor/SD_DAT2: track 0.00 -> 3.09 mm
- net /Power Measurement/I2C_SDA: track 119.2 -> 120.8 mm
- net /Microprocessor/SD_CS: track 27.4 -> 28.1 mm, vias 2 -> 3
- net +3.3V: track 78.7 -> 78.5 mm, vias 31 -> 30
- net /Microprocessor/SPI_COPI: vias 3 -> 4
Other:
- board text added: "BOOT G2"
- board text added: "ESP32-C3FH4 sensor board v0.3 Prototype - 2024-Oct-17"
- board text added: "EXT1 GPIO03 ADC"
- board text added: "Load Cell"
- board text added: "RX - G20"
- board text added: "SCL - G5"
- board text added: "SD DET - G11 CS - G14 SCK - G15 COPI - G16 CIPO - G17"
- board text added: "SD PU"
- board text added: "SDA - G4"
- board text added: "TX - G21"
- board text removed: "DET - GPIO11 CS - GPIO14"
- board text removed: "ESP32-C3FH4 sensor board v0.3 Prototype - 2024-Jul-18"
- board text removed: "EXT1 GPIO03-ADC"
- board text removed: "RX"
- board text removed: "SCK: GPIO15 COPI: GPIO16 CIPO: GPIO17"
- board text removed: "SCL"
- board text removed: "SDA"
- board text removed: "TX"
