File: hardware/v0/esp32_sensor_board/esp32_sensor_board.kicad_pcb (KiCad board)
At the start: 4 copper layers, 76 x 62 mm, 90 parts, among them J101 Conn_01x02, J102 Conn_01x02, J103 Conn_01x02, J104 Conn_01x02, J201 3.3V, J301 USB4510-03-1-A_REVA, J302 Micro_SD_Card_Det, J303 Conn_Coaxial, J304 UART, J305 EXT1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

Commit message: Revisions for recordering
Parts:
- removed J301: USB4510-03-1-A_REVA, USB4510-03-1-A:GCT_USB4510-03-1-A_REVA
- added J309: USB_C_Receptacle_USB2.0_16P, Connector_USB:USB_C_Receptacle_GCT_USB4085, F.Cu at (128.1, 76.3)
- added R313: 33R, Resistor_SMD:R_0603_1608Metric, F.Cu at (137.5, 76.0)
- moved C315 10.9 mm to (137.5, 74.0), turned to 180 degrees
Routing:
- net Net-(J302-VDD): track 0.00 -> 11.5 mm
- net +5V: track 16.9 -> 25.5 mm
- net +3.3V: track 78.5 -> 75.7 mm
- net /Microprocessor/USB_P: track 17.8 -> 20.3 mm
- net /Microprocessor/USB_N: track 21.8 -> 20.9 mm, vias 2 -> 1
- net GND: track 132.3 -> 132.2 mm, vias 70 -> 69
Other:
- outline, holes or cut-outs redrawn
- board text added: "ESP32-C3FH4 sensor board v0.4 Prototype - 2025-Jan-11"
- board text removed: "ESP32-C3FH4 sensor board v0.3 Prototype - 2024-Oct-17"
