File: hardware/v1 - S3 - Mic Focus/s3_sensor_board/esp32_sensor_power.kicad_sch (KiCad schematic)
At the start: 16 parts, among them J201 3.3V, U201 LMR36006

Commit message: WIP
Parts:
- renumbered D1 to D201, R203 to R201, R201 to R202, R202 to R203
Other:
- moved on the sheet: C201, C202, C203, C204, C205, C206, C207, C208, D201, JP201, L201, R202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
