File: hardware/v1 - S3 - Mic Focus/s3_sensor_board/sensor_loadcell.kicad_sch (KiCad schematic)
At the start: 9 parts, among them J501 Conn_01x05, J502 Conn_01x05

Commit message: WIP
Parts:
- renumbered C501 to C401, C502 to C402, C503 to C403, C504 to C404, C505 to C405, C506 to C406, J501 to J401, J502 to J402, U501 to U401
Changed lines of the file:
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@@
 		(dnp no)
 		(fields_autoplaced yes)
-		(property "Reference" "J502"
+		(property "Reference" "J402"
 			(at 38.1 100.33 0)
 			(show_name no)
@@
 			(project "s3_sensor_board"
 				(path "/d76badc5-1f0d-4fe6-889f-ca56408e093d/7fbfe679-89cc-4470-a0bc-43ba7c1b816f"
-					(reference "J502")
+					(reference "J402")
 					(unit 1)
 				)
@@
 		(dnp no)
 		(fields_autoplaced yes)
-		(property "Reference" "C505"
+		(property "Reference" "C405"
 			(at 45.72 171.4563 0)
 			(show_name no)
@@
 			(project "s3_sensor_board"
 				(path "/d76badc5-1f0d-4fe6-889f-ca56408e093d/7fbfe679-89cc-4470-a0bc-43ba7c1b816f"
-					(reference "C505")
+					(reference "C405")
 					(unit 1)
 				)
@@
 		(dnp no)
 		(fields_autoplaced yes)
-		(property "Reference" "#PWR0503"
+		(property "Reference" "#PWR0403"
 			(at 38.1 69.85 0)
 			(hide yes)
@@
 			(project "s3_sensor_board"
 				(path "/d76badc5-1f0d-4fe6-889f-ca56408e093d/7fbfe679-89cc-4470-a0bc-43ba7c1b816f"
-					(reference "#PWR0503")
+					(reference "#PWR0403")
 					(unit 1)
 				)
@@
 		(dnp no)
 		(fields_autoplaced yes)
-		(property "Reference" "C506"
+		(property "Reference" "C406"
 			(at 60.96 171.4563 0)
 			(show_name no)
@@
 			(project "s3_sensor_board"
 				(path "/d76badc5-1f0d-4fe6-889f-ca56408e093d/7fbfe679-89cc-4470-a0bc-43ba7c1b816f"
-					(reference "C506")
+					(reference "C406")
 					(unit 1)
 				)
@@
 		(dnp no)
 		(fields_autoplaced yes)
-		(property "Reference" "#PWR0507"
+		(property "Reference" "#PWR0407"
 			(at 129.54 123.19 0)
 			(hide yes)
@@
 			(project "s3_sensor_board"
 				(path "/d76badc5-1f0d-4fe6-889f-ca56408e093d/7fbfe679-89cc-4470-a0bc-43ba7c1b816f"
-					(reference "#PWR0507")
+					(reference "#PWR0407")
 					(unit 1)
 				)
@@
 		(dnp no)
 		(fields_autoplaced yes)
-		(property "Reference" "C504"
+		(property "Reference" "C404"
 			(at 144.78 102.8763 0)
 			(show_name no)
@@
 			(project "s3_sensor_board"
 				(path "/d76badc5-1f0d-4fe6-889f-ca56408e093d/7fbfe679-89cc-4470-a0bc-43ba7c1b816f"
-					(reference "C504")
+					(reference "C404")
 					(unit 1)
 				)
@@
 		(dnp no)
 		(fields_autoplaced yes)
-		(property "Reference" "#PWR0508"
+		(property "Reference" "#PWR0408"
 			(at 109.22 130.81 0)
 			(hide yes)
@@
 			(project "s3_sensor_board"
 				(path "/d76badc5-1f0d-4fe6-889f-ca56408e093d/7fbfe679-89cc-4470-a0bc-43ba7c1b816f"
-					(reference "#PWR0508")
+					(reference "#PWR0408")
 					(unit 1)
 				)
@@
 		(dnp no)
 		(fields_autoplaced yes)
-		(property "Reference" "C501"
+		(property "Reference" "C401"
 			(at 27.94 26.6763 0)
 			(show_name no)
@@
 			(project "s3_sensor_board"
 				(path "/d76badc5-1f0d-4fe6-889f-ca56408e093d/7fbfe679-89cc-4470-a0bc-43ba7c1b816f"
-					(reference "C501")
+					(reference "C401")
 					(unit 1)
 				)
@@
 		(dnp no)
 		(fields_autoplaced yes)
-		(property "Reference" "#PWR0506"
+		(property "Reference" "#PWR0406"
 			(at 111.76 82.55 0)
 			(hide yes)
@@
 			(project "s3_sensor_board"
 				(path "/d76badc5-1f0d-4fe6-889f-ca56408e093d/7fbfe679-89cc-4470-a0bc-43ba7c1b816f"
-					(reference "#PWR0506")
+					(reference "#PWR0406")
 					(unit 1)
 				)
@@
 		(dnp no)
 		(fields_autoplaced yes)
-		(property "Reference" "#PWR0505"
+		(property "Reference" "#PWR0405"
 			(at 76.2 69.85 0)
 			(hide yes)
@@
 			(project "s3_sensor_board"
 				(path "/d76badc5-1f0d-4fe6-889f-ca56408e093d/7fbfe679-89cc-4470-a0bc-43ba7c1b816f"
-					(reference "#PWR0505")
+					(reference "#PWR0405")
 					(unit 1)
 				)
@@
 		(dnp no)
 		(fields_autoplaced yes)
-		(property "Reference" "U501"
+		(property "Reference" "U401"
 			(at 115.2241 82.55 0)
 			(show_name no)
@@
 			(project "s3_sensor_board"
 				(path "/d76badc5-1f0d-4fe6-889f-ca56408e093d/7fbfe679-89cc-4470-a0bc-43ba7c1b816f"
-					(reference "U501")
+					(reference "U401")
 					(unit 1)
 				)
@@
 		(dnp no)
 		(fields_autoplaced yes)
-		(property "Reference" "#PWR0502"
+		(property "Reference" "#PWR0402"
 			(at 25.4 39.37 0)
 			(hide yes)
@@
 			(project "s3_sensor_board"
 				(path "/d76badc5-1f0d-4fe6-889f-ca56408e093d/7fbfe679-89cc-4470-a0bc-43ba7c1b816f"
-					(reference "#PWR0502")
+					(reference "#PWR0402")
 					(unit 1)
 				)
@@
 		(dnp no)
 		(fields_autoplaced yes)
-		(property "Reference" "C503"
+		(property "Reference" "C403"
 			(at 40.64 57.1563 0)
 			(show_name no)
@@
 			(project "s3_sensor_board"
 				(path "/d76badc5-1f0d-4fe6-889f-ca56408e093d/7fbfe679-89cc-4470-a0bc-43ba7c1b816f"
-					(reference "C503")
+					(reference "C403")
 					(unit 1)
 				)
@@
 		(dnp no)
 		(fields_autoplaced yes)
-		(property "Reference" "#PWR0504"
+		(property "Reference" "#PWR0404"
 			(at 60.96 69.85 0)
 			(hide yes)
@@
 			(project "s3_sensor_board"
 				(path "/d76badc5-1f0d-4fe6-889f-ca56408e093d/7fbfe679-89cc-4470-a0bc-43ba7c1b816f"
-					(reference "#PWR0504")
+					(reference "#PWR0404")
 					(unit 1)
 				)
@@
 		(dnp no)
 		(fields_autoplaced yes)
-		(property "Reference" "C502"
+		(property "Reference" "C402"
 			(at 30.48 57.1563 0)
 			(show_name no)
@@
 			(project "s3_sensor_board"
 				(path "/d76badc5-1f0d-4fe6-889f-ca56408e093d/7fbfe679-89cc-4470-a0bc-43ba7c1b816f"
-					(reference "C502")
+					(reference "C402")
 					(unit 1)
 				)
@@
 		(dnp no)
 		(fields_autoplaced yes)
-		(property "Reference" "#PWR0501"
+		(property "Reference" "#PWR0401"
 			(at 25.4 26.67 0)
 			(hide yes)
@@
 			(project "s3_sensor_board"
 				(path "/d76badc5-1f0d-4fe6-889f-ca56408e093d/7fbfe679-89cc-4470-a0bc-43ba7c1b816f"
-					(reference "#PWR0501")
+					(reference "#PWR0401")
 					(unit 1)
 				)
@@
 		(dnp no)
 		(fields_autoplaced yes)
-		(property "Reference" "J501"
+		(property "Reference" "J401"
 			(at 38.1 80.01 0)
 			(show_name no)
@@
 			(project "s3_sensor_board"
 				(path "/d76badc5-1f0d-4fe6-889f-ca56408e093d/7fbfe679-89cc-4470-a0bc-43ba7c1b816f"
-					(reference "J501")
-					(unit 1)
-				)
+					(reference "J401")
+					(unit 1)
+				)

Commit message: WIP
Parts:
- removed C406: DNP, Capacitor_SMD:C_0805_2012Metric, symbol Device:C_Small
- removed J402: Conn_01x05, Connector_PinHeader_2.54mm:PinHeader_1x05_P2.54mm_Horizontal, symbol Connector_Generic:Conn_01x05

Commit message: Processor placement and routing work
Parts:
- J401: footprint Connector_PinHeader_2.54mm:PinHeader_1x05_P2.54mm_Horizontal -> Connector_PinHeader_2.54mm:PinHeader_1x05_P2.54mm_Vertical
Changed lines of the file:
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@@
 			)
 		)
-		(property "Footprint" "Connector_PinHeader_2.54mm:PinHeader_1x05_P2.54mm_Horizontal"
+		(property "Footprint" "Connector_PinHeader_2.54mm:PinHeader_1x05_P2.54mm_Vertical"
 			(at 38.1 91.44 0)
 			(hide yes)
@@
 			(at 38.1 91.44 0)
 			(hide yes)
+			(show_name no)
+			(do_not_autoplace no)
+			(effects
+				(font
+					(size 1.27 1.27)
+				)
+			)
+		)
+		(property "MPN" ""
+			(at 38.1 91.44 0)
+			(hide yes)
