File: hardware/v1 - S3 - Mic Focus/s3_sensor_board/esp32_uc.kicad_sch (KiCad schematic)
At the start: 47 parts, among them J302 Micro_SD_Card_Det, J303 Conn_Coaxial, J304 UART, J305 EXT1, J306 EXT2, J307 I2C, J308 SPI, J309 USB_C_Receptacle_USB2.0_16P, SW301 BOOT, SW302 RST, U302 ESP32-C3, Y301 32kHz RTC Crystal, Y302 40 MHz

Commit message: v1 board started
Parts:
- removed U302: ESP32-C3, Package_DFN_QFN:QFN-32-1EP_5x5mm_P0.5mm_EP3.45x3.45mm, symbol Espressif:ESP32-C3
- added U1: ESP32-S3, Package_DFN_QFN:QFN-56-1EP_7x7mm_P0.4mm_EP4x4mm, symbol BVH Symbols:ESP32-S3
Connections:
- new net: U1.2 (VDD3P3), U1.3 (VDD3P3)
- new net: U1.55 (VDDA), U1.56 (VDDA)
- no-connect marks 5 -> 4
Other:
- note removed: "These pins are used for the internal flash and cannot be used for external SPI or SD card."

Commit message: WIP
Parts:
- removed J303: Conn_Coaxial, Connector_Coaxial:U.FL_Molex_MCRF_73412-0110_Vertical, symbol Connector:Conn_Coaxial
- removed J308: SPI, Connector_PinHeader_2.54mm:PinHeader_1x06_P2.54mm_Vertical, symbol Connector_Generic:Conn_01x06
- removed L301: 2.0nH, Inductor_SMD:L_0402_1005Metric, symbol Device:L_Small
- removed U303: (no value), BVH_Components_Misc:Diode_10Pin_DFN2510A-10_10-XFDFN_SOT1176-1, symbol BVH_Protection:PUSB3AB4
- added AE401: ANT, BVH_RF_Ham:ANT2012LL13R2400A, symbol BVH_RF_Ham:Antenna_Shield
- added C409, C410: DNP, Capacitor_SMD:C_0603_1608Metric, symbol Device:C_Small
- added FB401: (no value), Resistor_SMD:R_0805_2012Metric, symbol Device:FerriteBead_Small
- added J405: Conn_Coaxial, Connector_Coaxial:U.FL_Molex_MCRF_73412-0110_Vertical, symbol Connector:Conn_Coaxial
- added JP401: RF Ant Sel, BVH_Components_Misc:Jumper_Resistor_0603_2_Way, symbol Jumper:SolderJumper_3_Open
- added R408, R409, R410, R413, R415: 50k, Resistor_SMD:R_0603_1608Metric, symbol Device:R_Small
- added R411, R412: 0, Resistor_SMD:R_0603_1608Metric, symbol Device:R_Small
- R303: value R_Small -> 100k
Connections:
- net +3.3V: now also U1.2 (VDD3P3), U1.20 (VDD3P3_RTC), U1.3 (VDD3P3), U1.46 (VDD3P3_CPU), FB401.2, R408.2, R409.1, R410.2, R413.2, R415.2
- net CHIP_EN: now also U1.4 (CHIP_PU)
- net GND: now also AE401.2 (GND), C409.2, C410.2, J405.2 (Ext); no longer J302.8 (DAT1)
- net GPIO08_BOOT: no longer R301.1
- net I2C_SCK: now also U1.24 (GPIO18)
- net I2C_SDA: now also U1.23 (GPIO17)
- net RF: now also U1.1 (LNA_IN)
- net RF_ANT: now also JP401.2 (C)
- net SD_DAT2: now also U1.49 (GPIO43/U0TXD), R413.1
- net SD_DET: now also U1.50 (GPIO44/U0RXD)
- net SPI_CIPO: no longer J302.7 (DAT0)
- net SPI_COPI: no longer J302.3 (CMD)
- net SPI_SCK: no longer J302.5 (CLK)
- net STATUS_LED: now also U1.51 (GPIO45)
- net USB_N: now also C409.1, R411.1
- net USB_P: now also C410.1, R412.1
- net VDD33A: now also U1.55 (VDDA), U1.56 (VDDA), FB401.1
- net XTAL_32K_N: now also U1.22 (GPIO16/XTAL_32K_N*)
- net XTAL_32K_P: now also U1.21 (GPIO15/XTAL_32K_P*)
- net XTAL_N: now also U1.53 (XTAL_N)
- net XTAL_P: now also U1.54 (XTAL_P)
- net ADC1_4: now reaches U1.10 (GPIO5)
- net ADC1_5: now reaches U1.11 (GPIO6)
- net ADC1_6: now reaches U1.12 (GPIO7)
- net ADC1_7: now reaches U1.13 (GPIO8)
- net ADC1_8: now reaches U1.14 (GPIO9)
- net ADC1_9: now reaches U1.15 (GPIO10)
- net USB_uC_N: now reaches U1.25 (GPIO19/USB_D-)
- net USB_uC_N: now also R411.2
- net USB_uC_P: now reaches U1.26 (GPIO20/USB_D+)
- net USB_uC_P: now also R412.2
- net SD_DAT1: now reaches U1.43 (GPIO38)
- net SD_DAT1: now also J302.8 (DAT1), R410.1
- net SD_DAT0: now reaches U1.44 (GPIO39/MTCK)
- net SD_DAT0: now also J302.7 (DAT0), R408.1
- net SD_SCK: now reaches U1.45 (GPIO40/MTDO)
- net SD_SCK: now also J302.5 (CLK)
- net SD_CMD: now reaches U1.47 (GPIO41/MTDI)
- net SD_CMD: now also J302.3 (CMD), R409.2
- net SD_DAT3: now reaches U1.48 (GPIO42/MTMS)
- net SD_DAT3: now also R415.1
- net BOOT_MODE: now reaches U1.5 (GPIO0)
- net ADC1_0: now reaches U1.6 (GPIO1)
- net ADC1_1: now reaches U1.7 (GPIO2)
- net GPIO3_STRAP_PD: now reaches U1.8 (GPIO3)
- net GPIO3_STRAP_PD: now also R301.1
- net ADC1_3: now reaches U1.9 (GPIO4)
- net +5V renamed V_usb
- new net: AE401.1 (A), JP401.1 (A)
- new net: J405.1 (In), JP401.3 (B)
- no-connect marks 4 -> 14
Other:
- note removed: "DNP"
- note removed: "SD card and SPI bus are mutually exclusive. For SPI bus, DNP SD Card PU resistors"
- moved on the sheet: C307, C308, C309, C310, C311, C312, C313, C314, L302, R301, R302, R303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

Commit message: WIP
Parts:
- removed J305: EXT1, Connector_PinHeader_2.54mm:PinHeader_1x03_P2.54mm_Vertical, symbol Connector:Conn_01x03_Socket
- removed J306: EXT2, Connector_PinHeader_2.54mm:PinHeader_1x03_P2.54mm_Vertical, symbol Connector:Conn_01x03_Socket
- SW301: footprint BVH_Switches:TacButton_SMD_5mm_5mm -> BVH_Switches:TacButton_SMD_4.0x3.0mm_SPST_NO_2P
- SW302: footprint BVH_Switches:Tac_SMD_6.4mm_Side_SPST_NO -> BVH_Switches:TacButton_SMD_4.0x3.0mm_SPST_NO_2P
- renumbered AE401 to AE301, C307 to C305, C305 to C306, C306 to C307, C409 to C309, C410 to C310, C315 to C311, C313 to C312, C314 to C313, C309 to C314, C310 to C315, C311 to C316, C312 to C317, FB401 to FB301, J304 to J301, J307 to J302, J309 to J303, J405 to J304, J302 to J305, JP401 to JP301, L302 to L301, R306 to R301, R301 to R302, R302 to R303, R311 to R304, R312 to R305, R303 to R306, R308 to R307, R314 to R308, R411 to R309, R412 to R310, R307 to R311, R310 to R312, R309 to R313, R313 to R314, R408 to R315, R409 to R316, R410 to R317, R413 to R318, R415 to R319, R304 to R320, R305 to R321, U1 to U302
Connections:
- net SD_CMD: now also U302.41 (GPIO36); no longer U302.47 (GPIO41/MTDI)
- net SD_DAT0: now also U302.39 (GPIO34); no longer U302.44 (GPIO39/MTCK)
- net SD_DAT1: now also U302.38 (GPIO33); no longer U302.43 (GPIO38)
- net SD_DAT2: now also U302.43 (GPIO38); no longer U302.49 (GPIO43/U0TXD)
- net SD_DAT3: now also U302.42 (GPIO37); no longer U302.48 (GPIO42/MTMS)
- net SD_DET: now also U302.44 (GPIO39/MTCK); no longer U302.50 (GPIO44/U0RXD)
- net SD_SCK: now also U302.40 (GPIO35); no longer U302.45 (GPIO40/MTDO)
- net UART_RX: now also U302.50 (GPIO44/U0RXD)
- net UART_TX: now also U302.49 (GPIO43/U0TXD)
- net PDM_D0: now reaches U302.16 (GPIO11)
- net PDM_D1: now reaches U302.17 (GPIO12)
- net PDM_D2: now reaches U302.18 (GPIO13)
- net PDM_D3: now reaches U302.19 (GPIO14)
- net ADC1_0 renamed Vin_DIV
- net ADC1_1: no longer names the net of U302.7 (GPIO2)
- net ADC1_3: no longer names the net of U302.9 (GPIO4)
- net ADC1_4: no longer names the net of U302.10 (GPIO5)
- net ADC1_5: no longer names the net of U302.11 (GPIO6)
- net ADC1_6: no longer names the net of U302.12 (GPIO7)
- net ADC1_7: no longer names the net of U302.13 (GPIO8)
- net ADC1_8: no longer names the net of U302.14 (GPIO9)
- net ADC1_9 renamed PDM_CLK
Other:
- moved on the sheet: J302, R309

Commit message: WIP
Parts:
- removed R307, R308, R311, R312, R313: 50k, Resistor_SMD:R_0603_1608Metric, symbol Device:R_Small
- R309: renamed from R314; value 33R -> 0R
- renumbered R302 to R301, R303 to R302, R301 to R303, R309 to R307, R310 to R308, R315 to R310, R316 to R311, R317 to R312, R318 to R313, R319 to R314, R320 to R315, R321 to R316
Connections:
- net SD_CS is gone; now on net SD_DAT3: J305.2 (DAT3/CD)
- net DATA_READY: now also U302.27 (GPIO21)
- net GND: now also U302.57 (GND)
- net GPIO09_BOOT: now also U302.14 (GPIO9)
- net I2C_SCK: now also U302.42 (GPIO37); no longer U302.24 (GPIO18)
- net I2C_SDA: now also U302.43 (GPIO38); no longer U302.23 (GPIO17)
- net SD_CMD: now also U302.49 (GPIO43/U0TXD); no longer U302.41 (GPIO36)
- net SD_DAT0: now also U302.47 (GPIO41/MTDI); no longer U302.39 (GPIO34)
- net SD_DAT1: now also U302.45 (GPIO40/MTDO); no longer U302.38 (GPIO33)
- net SD_DAT2: now also U302.51 (GPIO45); no longer U302.43 (GPIO38)
- net SD_DAT3: now also U302.50 (GPIO44/U0RXD); no longer U302.42 (GPIO37)
- net SD_DET: now also U302.52 (GPIO46); no longer U302.44 (GPIO39/MTCK)
- net SD_SCK: now also U302.48 (GPIO42/MTMS); no longer U302.40 (GPIO35)
- net STATUS_LED: no longer U302.51 (GPIO45)
- net UART_RX: no longer U302.50 (GPIO44/U0RXD)
- net UART_TX: no longer U302.49 (GPIO43/U0TXD)
- net XTAL_32K_P_R: now reaches C314.1, R315.2, Y301.1
- net SD_VDD: now reaches J305.4 (VDD), R309.2
- net XTAL_P_R: now reaches C316.1, R316.2, Y302.1
Other:
- moved on the sheet: D301, J301, J302, J303, R303, R304, R305, R316, U301

Commit message: Processor placement and routing work
Connections:
- net DATA_READY: now also U302.44 (GPIO39/MTCK); no longer U302.27 (GPIO21)
Changed lines of the file:
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@@
 	(hierarchical_label "DATA_READY"
 		(shape input)
-		(at 100.33 115.57 180)
+		(at 152.4 104.14 0)
 		(effects
 			(font
 				(size 1.27 1.27)
 			)
-			(justify right)
+			(justify left)
 		)
 	)

Commit message: WIP
Parts:
- R303: value R_Small -> 1k
Changed lines of the file:
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@@
 			)
 		)
-		(property "Value" "R_Small"
+		(property "Value" "1k"
 			(at 264.16 48.26 90)
 			(show_name no)
@@
 			(at 264.16 50.8 0)
 			(hide yes)
+			(show_name no)
+			(do_not_autoplace no)
+			(effects
+				(font
+					(size 1.27 1.27)
+				)
+			)
+		)
+		(property "MPN" ""
+			(at 264.16 50.8 0)
+			(hide yes)

Commit message: WIP
Parts:
- removed J301: UART, Connector_PinHeader_2.54mm:PinHeader_1x03_P2.54mm_Vertical, symbol Connector:Conn_01x03_Socket
- removed J302: I2C, Connector_PinHeader_2.54mm:PinHeader_1x04_P2.54mm_Vertical, symbol Connector:Conn_01x04_Socket
Connections:
- net SD_CMD: now also U302.48 (GPIO42/MTMS); no longer U302.49 (GPIO43/U0TXD)
- net SD_DAT0: now also U302.50 (GPIO44/U0RXD); no longer U302.47 (GPIO41/MTDI)
- net SD_DAT1: now also U302.51 (GPIO45); no longer U302.45 (GPIO40/MTDO)
- net SD_DAT2: now also U302.45 (GPIO40/MTDO); no longer U302.51 (GPIO45)
- net SD_DAT3: now also U302.47 (GPIO41/MTDI); no longer U302.50 (GPIO44/U0RXD)
- net SD_SCK: now also U302.49 (GPIO43/U0TXD); no longer U302.48 (GPIO42/MTMS)
