File: hardware/v1 - S3 - Mic Focus/s3_sensor_board/esp32_uc.kicad_sch (KiCad schematic)
At the start: 47 parts, among them J303 USB_C_Receptacle_USB2.0_16P, J304 Conn_Coaxial, J305 Micro_SD_Card_Det, SW301 BOOT, SW302 RST, U302 ESP32-S3, Y301 32kHz RTC Crystal, Y302 40 MHz

Commit message: Layout, starting DRC
Parts:
- removed R302: 100k, Resistor_SMD:R_0603_1608Metric, symbol Device:R_Small
- renumbered J303 to J301, J304 to J302, J305 to J303, R303 to R302, R304 to R303, R305 to R304, R306 to R305, R307 to R306, R308 to R307, R309 to R308, R310 to R309, R311 to R310
Connections:
- net BOOT_MODE: now also SW301.1 (A)
- net DATA_READY: now also U302.42 (GPIO37); no longer U302.44 (GPIO39/MTCK)
- net I2C_SCK: now also U302.40 (GPIO35); no longer U302.42 (GPIO37)
- net I2C_SDA: now also U302.41 (GPIO36); no longer U302.43 (GPIO38)
- net SD_CMD: now also U302.47 (GPIO41/MTDI); no longer U302.48 (GPIO42/MTMS)
- net SD_DAT0: now also U302.49 (GPIO43/U0TXD); no longer U302.50 (GPIO44/U0RXD)
- net SD_DAT1: now also U302.50 (GPIO44/U0RXD); no longer U302.51 (GPIO45)
- net SD_DAT2: now also U302.44 (GPIO39/MTCK); no longer U302.45 (GPIO40/MTDO)
- net SD_DAT3: now also U302.45 (GPIO40/MTDO); no longer U302.47 (GPIO41/MTDI)
- net SD_DET: now also U302.43 (GPIO38); no longer U302.52 (GPIO46)
- net SD_SCK: now also U302.48 (GPIO42/MTMS); no longer U302.49 (GPIO43/U0TXD)
- net STATUS_LED: now also U302.52 (GPIO46)
- net GPIO09_BOOT: no longer names the net of U302.14 (GPIO9)
- net GPIO09_BOOT: no longer SW301.1 (A)
- no-connect marks 14 -> 15
Other:
- moved on the sheet: R301, Reference: SW301

Commit message: S3 WIP - Initial submission
Connections:
- net RF_ANT_CONN: now reaches AE301.1 (A), JP301.1 (A)
- net RF_ANT_CHIP: now reaches J302.1 (In), JP301.3 (B)
Changed lines of the file:
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@@
 	)
 	(junction
+		(at 49.53 132.08)
+		(diameter 0)
+		(color 0 0 0 0)
+	)
+	(junction
 		(at 208.28 125.73)
 		(diameter 0)
@@
 	(wire
 		(pts
+			(xy 49.53 132.08) (xy 49.53 133.35)
+		)
+		(stroke
+			(width 0)
+			(type default)
+		)
+	)
+	(wire
+		(pts
 			(xy 190.5 160.02) (xy 193.04 160.02)
 		)
@@
 	(wire
 		(pts
-			(xy 49.53 130.81) (xy 49.53 133.35)
+			(xy 49.53 130.81) (xy 49.53 132.08)
 		)
 		(stroke
@@
 	(wire
 		(pts
+			(xy 46.99 132.08) (xy 49.53 132.08)
+		)
+		(stroke
+			(width 0)
+			(type default)
+		)
+	)
+	(wire
+		(pts
 			(xy 91.44 185.42) (xy 99.06 185.42)
 		)
@@
 		)
 	)
+	(label "RF_ANT_CONN"
+		(at 46.99 132.08 90)
+		(effects
+			(font
+				(size 1.27 1.27)
+			)
+			(justify left bottom)
+		)
+	)
 	(label "SD_DET"
 		(at 237.49 158.75 180)
@@
 		)
 	)
+	(label "RF_ANT_CHIP"
+		(at 49.53 146.05 270)
+		(effects
+			(font
+				(size 1.27 1.27)
+			)
+			(justify right bottom)
+		)
+	)
 	(label "USB_P"
 		(at 251.46 97.79 0)
@@
 		)
 	)
-	(netclass_flag ""
-		(length 2.54)
-		(shape round)
-		(at 49.53 146.05 180)
-		(fields_autoplaced yes)
-		(effects
-			(font
-				(size 1.27 1.27)
-			)
-			(justify right bottom)
-		)
-		(property "Netclass" "50ohm"
-			(at 50.2285 148.59 0)
-			(show_name no)
-			(do_not_autoplace no)
-			(effects
-				(font
-					(size 1.27 1.27)
-				)
-				(justify left)
-			)
-		)
-		(property "Component Class" ""
-			(at -17.78 -20.32 0)
-			(show_name no)
-			(do_not_autoplace no)
-			(effects
-				(font
-					(size 1.27 1.27)
-					(italic yes)
-				)
-			)
-		)
-	)
-	(netclass_flag ""
-		(length 2.54)
-		(shape round)
-		(at 49.53 132.08 90)
-		(fields_autoplaced yes)
-		(effects
-			(font
-				(size 1.27 1.27)
-			)
-			(justify left bottom)
-		)
-		(property "Netclass" "50ohm"
-			(at 46.99 131.3815 90)
-			(show_name no)
-			(do_not_autoplace no)
-			(effects
-				(font
-					(size 1.27 1.27)
-				)
-				(justify left)
-			)
-		)
-		(property "Component Class" ""
-			(at -17.78 -34.29 0)
-			(show_name no)
-			(do_not_autoplace no)
-			(effects
-				(font
-					(size 1.27 1.27)
-					(italic yes)
-				)
-			)
-		)
-	)
