File: hardware/v1 - S3 - Mic Focus/s3_sensor_board/s3_sensor_board.kicad_pcb (KiCad board)
At the start: 4 copper layers, 20 x 100 mm, 76 parts, among them J101 Conn_01x02, J102 PWR, J103 EXP, J301 UART, J302 I2C, J303 USB_C_Receptacle_USB2.0_16P, J304 Conn_Coaxial, J305 Micro_SD_Card_Det, SW301 BOOT, SW302 RST, U201 TPS564257DRLR, U302 ESP32-S3, U501 SHT4x, Y301 32kHz RTC Crystal, Y302 40 MHz

Commit message: WIP
Parts:
- removed J301: UART, Connector_PinHeader_2.54mm:PinHeader_1x03_P2.54mm_Vertical
- removed J302: I2C, Connector_PinHeader_2.54mm:PinHeader_1x04_P2.54mm_Vertical
- J103: moved to B.Cu
- moved D301 72.9 mm to (117.6, 116.2)
- moved R303 72.9 mm to (117.3, 114.2)
- moved C501 66.3 mm to (149.1, 122.1), turned to -90 degrees
- moved U501 62.3 mm to (147.0, 122.0), turned to 90 degrees
- moved SW302 35.4 mm to (156.5, 99.8), turned to 180 degrees
- moved SW301 34.5 mm to (156.5, 96.8), turned to 0 degrees
- moved J103 23.9 mm to (155.6, 130.8), turned to 90 degrees
- moved R101 8.02 mm to (141.5, 86.0)
- moved R102 8.02 mm to (141.5, 89.2)
- moved C303 0.82 mm to (148.5, 96.8)
Connections:
- U302 pad 45: /Microprocessor/SD_DAT1 -> /Microprocessor/SD_DAT2
- U302 pad 47: /Microprocessor/SD_DAT0 -> /Microprocessor/SD_DAT3
- U302 pad 48: /Microprocessor/SD_SCK -> /Microprocessor/SD_CMD
- U302 pad 49: /Microprocessor/SD_CMD -> /Microprocessor/SD_SCK
- U302 pad 50: /Microprocessor/SD_DAT3 -> /Microprocessor/SD_DAT0
- U302 pad 51: /Microprocessor/SD_DAT2 -> /Microprocessor/SD_DAT1
Routing:
- net /Microprocessor/SD_DAT1: track 0.00 -> 50.7 mm, vias 0 -> 1
- net /Microprocessor/SD_DAT0: track 0.00 -> 48.3 mm, vias 0 -> 1
- net /Microprocessor/SD_CMD: track 0.00 -> 45.2 mm, vias 0 -> 1
- net /Microprocessor/SD_DAT3: track 0.00 -> 44.0 mm, vias 0 -> 1
- net /Microprocessor/SD_DAT2: track 0.00 -> 43.3 mm, vias 0 -> 1
- net /Microprocessor/SD_SCK: track 0.00 -> 39.4 mm, vias 0 -> 1
- net /PDM_D1: track 0.00 -> 37.4 mm, vias 0 -> 1
- net /Microprocessor/SD_DET: track 0.00 -> 36.7 mm, vias 0 -> 1
- net /PDM_D3: track 0.00 -> 35.7 mm, vias 0 -> 1
- net /I2C_SDA: track 0.00 -> 35.6 mm, vias 0 -> 1
- net /PDM_CLK: track 0.00 -> 35.0 mm, vias 0 -> 1
- net /PDM_D2: track 0.00 -> 33.8 mm, vias 0 -> 1
- net /PDM_D0: track 0.00 -> 33.0 mm, vias 0 -> 1
- net /I2C_SCL: track 0.00 -> 31.6 mm, vias 0 -> 1
- net /INT: track 0.00 -> 24.4 mm, vias 0 -> 1
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- added copper zone on B.Cu, net GND

Commit message: Layout, starting DRC
Parts:
- removed the R302 at (173.7, 105.3)
- moved H101 114.6 mm to (122.8, 109.0)
- moved H102 114.6 mm to (122.8, 116.2)
- moved H103 114.6 mm to (122.8, 123.3)
- moved H104 114.6 mm to (122.8, 130.5)
- moved R103 97.6 mm to (159.2, 139.4), turned to 90 degrees
- moved R104 94.7 mm to (157.8, 139.4), turned to 90 degrees
- moved SW301 58.9 mm to (144.5, 154.5), turned to -90 degrees
- moved SW302 54.7 mm to (156.5, 154.5), turned to 90 degrees
- moved R305 51.5 mm to (153.8, 152.8), turned to -90 degrees
- moved C308 50.6 mm to (151.8, 153.0), turned to -90 degrees
- moved R302 41.3 mm to (158.0, 121.5), turned to 180 degrees
- moved D301 40.8 mm to (157.8, 123.2)
- moved C306 23.5 mm to (154.2, 97.0), turned to 180 degrees
- moved C307 20.4 mm to (154.4, 98.8), turned to 180 degrees
- moved R301 18.6 mm to (154.5, 100.5)
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- renumbered J303 to J301, J304 to J302, J305 to J303, R303 to R302, R304 to R303, R305 to R304, R306 to R305, R307 to R306, R308 to R307, R309 to R308, R310 to R309, R311 to R310
Connections:
- J103 pad 2: +3V3 -> +3.3V
- SW301 pad 1: /Microprocessor/GPIO09_BOOT -> /Microprocessor/BOOT_MODE
- U302 pad 14: /Microprocessor/GPIO09_BOOT -> unconnected-(U302-GPIO9-Pad14)
- U302 pad 40: unconnected-(U302-GPIO35-Pad40) -> /I2C_SCL
- U302 pad 41: unconnected-(U302-GPIO36-Pad41) -> /I2C_SDA
- U302 pad 42: /I2C_SCL -> /INT
- U302 pad 43: /I2C_SDA -> /Microprocessor/SD_DET
- U302 pad 44: /INT -> /Microprocessor/SD_DAT2
- U302 pad 45: /Microprocessor/SD_DAT2 -> /Microprocessor/SD_DAT3
- U302 pad 47: /Microprocessor/SD_DAT3 -> /Microprocessor/SD_CMD
- U302 pad 48: /Microprocessor/SD_CMD -> /Microprocessor/SD_SCK
- U302 pad 49: /Microprocessor/SD_SCK -> /Microprocessor/SD_DAT0
- U302 pad 50: /Microprocessor/SD_DAT0 -> /Microprocessor/SD_DAT1
- U302 pad 51: /Microprocessor/SD_DAT1 -> unconnected-(U302-GPIO45-Pad51)
- U302 pad 52: /Microprocessor/SD_DET -> /Microprocessor/STATUS_LED
Routing:
- net +3.3V: track 31.8 -> 185.5 mm, vias 1 -> 11
- net /Microprocessor/BOOT_MODE: track 0.00 -> 69.9 mm, vias 0 -> 2
- net /Microprocessor/CHIP_EN: track 0.00 -> 64.1 mm, vias 0 -> 2
- net /Microprocessor/Vin_DIV: track 1.55 -> 23.8 mm, vias 0 -> 2
- net /Microprocessor/STATUS_LED: track 0.00 -> 22.2 mm, vias 0 -> 2
- net /TPS56425X Regulator/PWR_GD: track 2.07 -> 20.5 mm, vias 0 -> 1
- net /I2C_SCL: track 31.6 -> 49.5 mm
- net /I2C_SDA: track 35.6 -> 52.7 mm
- net /Microprocessor/GPIO3_STRAP_PD: track 0.00 -> 5.43 mm
- net GND: track 6.44 -> 3.33 mm, vias 12 -> 55
- net /Microprocessor/SD_DET: track 36.7 -> 35.0 mm
- net /Microprocessor/XTAL_32K_N: track 20.6 -> 19.0 mm
- net /Microprocessor/XTAL_32K_P: track 14.0 -> 12.8 mm
- net /TPS56425X Regulator/Vin: track 12.7 -> 11.7 mm
- net /Microprocessor/SD_DAT3: track 44.0 -> 43.3 mm
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- added copper zone on B.Cu, net +3.3V
