File: hardware/v1 - S3 - Mic Focus/s3_sensor_board/s3_sensor_board.kicad_pcb (KiCad board)
At the start: 4 copper layers, 20 x 100 mm, 73 parts, among them J101 Conn_01x02, J102 PWR, J103 EXP, J301 USB_C_Receptacle_USB2.0_16P, J302 Conn_Coaxial, J303 Micro_SD_Card_Det, SW301 BOOT, SW302 RST, U201 TPS564257DRLR, U302 ESP32-S3, U501 SHT4x, Y301 32kHz RTC Crystal, Y302 40 MHz

Commit message: S3 WIP - Initial submission
Parts:
- removed H103, H104: MountingHole_Pad, MountingHole:MountingHole_2.2mm_M2_DIN965_Pad
- moved H102 54.3 mm to (158.0, 157.5)
- moved H101 52.5 mm to (143.0, 157.5)
- moved C308 7.86 mm to (157.9, 148.1), turned to 90 degrees
- moved SW301 4.00 mm to (148.5, 154.5)
- moved SW302 4.00 mm to (152.5, 154.5)
- moved R305 3.02 mm to (156.5, 151.5), turned to 90 degrees
- moved C303 1.10 mm to (149.6, 96.8)
Connections:
- net Net-(AE301-A) renamed /Microprocessor/RF_ANT_CONN
- net Net-(J302-In) renamed /Microprocessor/RF_ANT_CHIP
Routing:
- net /TPS56425X Regulator/Vin: track 11.7 -> 29.6 mm
- net /Microprocessor/V_usb: track 6.74 -> 12.6 mm
- net /Microprocessor/BOOT_MODE: track 69.9 -> 64.1 mm
- net Net-(J301-CC1): track 0.00 -> 3.28 mm
- net +3.3V: track 185.5 -> 188.2 mm
- net /Microprocessor/RF_ANT_CONN: track 0.00 -> 1.83 mm
- net Net-(D301-A): track 0.00 -> 1.79 mm
- net /Microprocessor/CHIP_EN: track 64.1 -> 65.3 mm
- net /Microprocessor/SD_DAT1: track 50.3 -> 49.4 mm
- net /PDM_D0: track 33.0 -> 33.6 mm
- net /Microprocessor/SD_DAT2: track 43.2 -> 42.7 mm
- net GND: track 3.33 -> 2.99 mm, vias 55 -> 57

Commit message: WIP, standoffs
Parts:
- moved H101 0.71 mm to (143.5, 157.0)
- moved H102 0.71 mm to (157.5, 157.0)
Changed lines of the file:
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@@
 		(capping no)
 		(filling no)
-		(zone_defaults)
 		(grid_origin 140.5 60)
 		(pcbplotparams
@@
 	(footprint "MountingHole:MountingHole_2.2mm_M2_DIN965_Pad"
 		(layer "F.Cu")
-		(at 143 157.5)
+		(at 143.5 157)
 		(descr "Mounting Hole 2.2mm, M2, generated by kicad-footprint-generator mountinghole.py")
 		(tags "mountinghole M2 DIN965")
@@
 	(footprint "MountingHole:MountingHole_2.2mm_M2_DIN965_Pad"
 		(layer "F.Cu")
-		(at 158 157.5)
+		(at 157.5 157)
 		(descr "Mounting Hole 2.2mm, M2, generated by kicad-footprint-generator mountinghole.py")
 		(tags "mountinghole M2 DIN965")
@@
 	)
 	(segment
+		(start 156.233 116)
+		(end 156.233 113.042)
+		(width 0.34925)
+		(layer "F.Cu")
+		(net "/Microprocessor/RF_ANT_CHIP")
+	)
+	(segment
 		(start 149.025 79.35)
 		(end 149.67 78.705)
@@
 	)
 	(segment
+		(start 157.808 111.467)
+		(end 157.875 111.4)
+		(width 0.34925)
+		(layer "F.Cu")
+		(net "/Microprocessor/RF_ANT_CONN")
+	)
+	(segment
+		(start 157.808 113.2)
+		(end 157.808 111.467)
+		(width 0.34925)
+		(layer "F.Cu")
+		(net "/Microprocessor/RF_ANT_CONN")
+	)
+	(segment
 		(start 156.325 109.7375)
 		(end 157.8625 108.2)
@@
 		(net "/Microprocessor/V_usb")
 	)
-	(segment
-		(start 157.808 111.467)
-		(end 157.875 111.4)
-		(width 0.34925)
-		(layer "F.Cu")
-		(net "/Microprocessor/RF_ANT_CONN")
-	)
-	(segment
-		(start 157.808 113.2)
-		(end 157.808 111.467)
-		(width 0.34925)
-		(layer "F.Cu")
-		(net "/Microprocessor/RF_ANT_CONN")
-	)
-	(segment
-		(start 156.233 116)
-		(end 156.233 113.042)
-		(width 0.34925)
-		(layer "F.Cu")
-		(net "/Microprocessor/RF_ANT_CHIP")
-	)
 	(zone

Commit message: WIP Fanout Board
Parts:
- added G***: LOGO, BVH_Logos:SkyIron_logo_Back, F.Cu at (150.0, 77.0)
- moved J103 0.50 mm to (155.6, 131.3)
Routing:
- net /Microprocessor/SD_DAT2: track 42.7 -> 48.3 mm
- net /Microprocessor/BOOT_MODE: track 64.1 -> 65.9 mm
- net +3.3V: track 188.2 -> 189.3 mm
Other:
- board text added: "AB4EN ESP32-S3 Sensor Board 2026-Sep-24 v0"

Commit message: Standoff move, silkscreen work
Parts:
- moved H101 1.06 mm to (142.8, 157.8)
- moved H102 1.06 mm to (158.2, 157.8)
- moved G*** 1.00 mm to (151.0, 77.0)
Other:
- board text added: "${BOARD_DATE} - ${BOARD_REV}"
- board text added: "${BOARD_NAME}"
- board text added: "${OWNER}"
- board text added: "1-GND 2-3.3V 3-CLK-10 4-D0-11 5-D1-12 6-D2-13 7-D3-14 8-RDY-37 9-SCK-35 10-SDA-36"
- board text added: "D0-43 D2-39 D1-44 D3-40 SCK-42 CMD-41 DET-38"
- board text removed: "AB4EN ESP32-S3 Sensor Board 2026-Sep-24 v0"
