File: hardware/v1 - S3 - Mic Focus/pdm_fanout/pdm_fanout.kicad_pcb (KiCad board)
At the start: 2 copper layers, 20 x 100 mm, 12 parts, among them J1 D0_L, J2 D0_R, J3 D1_L, J4 D1_R, J5 D2_L, J6 D2_R, J7 D3_L, J8 D3_R, J9 EXP

Commit message: Standoff move, silkscreen work
Parts:
- moved H1 14.9 mm to (142.8, 157.8)
- moved G*** 14.2 mm to (150.8, 70.8), turned to 90 degrees
- moved H2 13.9 mm to (158.2, 157.8)
- moved J1 13.8 mm to (144.3, 87.0)
- moved J2 13.8 mm to (144.3, 82.4)
- moved J3 13.8 mm to (144.3, 97.5)
- moved J4 13.8 mm to (144.3, 92.9)
- moved J5 13.8 mm to (144.3, 108.0)
- moved J6 13.8 mm to (144.3, 103.4)
- moved J7 13.8 mm to (144.3, 119.6)
- moved J8 13.8 mm to (144.3, 115.0)
- moved J9 13.8 mm to (150.5, 130.0)
Routing:
- net GND: vias 12 -> 2
Other:
- board text added: "${BOARD_DATE} - ${BOARD_REV}"
- board text added: "${BOARD_NAME}"
- board text added: "${OWNER}"
- board text removed: "AB4EN ESP32-S3 Sensor Board PDM Microphone Fan-out 2026-Sep-24 v0"
