File: hardware/v1 - S3 - Mic Focus/pdm_fanout/pdm_fanout.kicad_sch (KiCad schematic)
At the start: 9 parts, among them J1 D0_L, J2 D0_R, J3 D1_L, J4 D1_R, J5 D2_L, J6 D2_R, J7 D3_L, J8 D3_R, J9 EXP

Commit message: WIP Fanout Board
Parts:
- added H1, H2: MountingHole_Pad, MountingHole:MountingHole_2.2mm_M2_DIN965_Pad, symbol Mechanical:MountingHole_Pad
- J1, J2, J3, J4, J5, J6, J7, J8: footprint (none) -> Connector_PinHeader_2.54mm:PinHeader_1x06_P2.54mm_Vertical; symbol Connector_Generic:Conn_01x05 -> Connector_Generic:Conn_01x06
- J9: footprint (none) -> BVH_Connectors_Misc:Conn_IDC_Female_Board_Mount_02x05_Abomination
Connections:
- net GND: now also J1.6 (Pin_6), J2.6 (Pin_6), J3.6 (Pin_6), J4.6 (Pin_6), J5.6 (Pin_6), J6.6 (Pin_6), J7.6 (Pin_6), J8.6 (Pin_6), H1.1, H2.1
Other:
- moved on the sheet: J9

Commit message: Standoff move, silkscreen work
Changed lines of the file:
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@@
-	)
-	(symbol
-		(lib_id "BVH Symbols:SkyIronLogo-Back")
-		(at 243.84 127 0)
-		(unit 1)
-		(body_style 1)
-		(exclude_from_sim no)
-		(in_bom yes)
-		(on_board yes)
-		(in_pos_files yes)
-		(dnp no)
-		(fields_autoplaced yes)
-		(property "Reference" "#LOGO1"
-			(at 243.84 121.92 0)
-			(show_name no)
-			(do_not_autoplace no)
-			(effects
-				(font
-					(size 1.27 1.27)
-				)
-			)
-		)
-		(property "Value" "SkyIronLogo-Back"
-			(at 243.84 124.46 0)
-			(show_name no)
-			(do_not_autoplace no)
-			(effects
-				(font
-					(size 1.27 1.27)
-				)
-			)
-		)
-		(property "Footprint" "BVH_Logos:SkyIron_logo_Back"
-			(at 243.84 124.46 0)
-			(hide yes)
-			(show_name no)
-			(do_not_autoplace no)
-			(effects
-				(font
-					(size 1.27 1.27)
-				)
-			)
-		)
-		(property "Datasheet" ""
-			(at 243.84 127 0)
-			(hide yes)
-			(show_name no)
-			(do_not_autoplace no)
-			(effects
-				(font
-					(size 1.27 1.27)
-				)
-			)
-		)
-		(property "Description" ""
-			(at 243.84 127 0)
-			(hide yes)
-			(show_name no)
-			(do_not_autoplace no)
-			(effects
-				(font
-					(size 1.27 1.27)
-				)
-			)
-		)
-		(instances
-			(project "pdm_fanout"
-				(path "/7d2357e8-908c-458b-9e6f-dadb8c3c2794"
-					(reference "#LOGO1")
-					(unit 1)
-				)
-			)
-		)
 	)
 	(symbol
